Commit message: [update] 调整双轮差速模型

File: src/description/urdf/diffbot_description.urdf.xacro (robot description, xacro)
@@ -4,22 +4,21 @@
         <!-- Constants for robot dimensions -->
         <xacro:property name="PI" value="3.1415926535897931"/>
+        <xacro:property name="SQRT_3" value="1.732050807568877"/>
         <!-- arbitrary value for base -->
-        <xacro:property name="base_mass" value="0.3" />
-        <xacro:property name="base_width" value="0.1" />
-        <xacro:property name="base_length" value="0.1" />
-        <xacro:property name="base_height" value="0.05" />
+        <xacro:property name="base_mass" value="5.0" />
+        <xacro:property name="base_len" value="0.100" />
+        <xacro:property name="base_radius" value="0.240" />
         <!-- arbitrary value for wheel -->
         <xacro:property name="wheel_mass" value="0.3" />
-        <xacro:property name="wheel_len" value="0.020" />
-        <xacro:property name="wheel_radius" value="0.015" />
+        <xacro:property name="wheel_len" value="0.050" />
+        <xacro:property name="wheel_radius" value="0.070" />
         <!-- arbitrary value for caster wheel -->
         <xacro:property name="caster_wheel_mass" value="0.1" />
-        <xacro:property name="caster_wheel_radius" value="0.015" />
         <!-- Space btw top of beam and the each joint -->
-        <xacro:property name="z_offset" value="-${base_height/2}" />
-        <xacro:property name="x_offset_head" value="${base_length/3}" />
-        <xacro:property name="x_offset_tail" value="-${base_length/3}" />
-        <!-- Foot Print -->
-        <link name="${prefix}base_footprint"/>
+        <xacro:property name="z_offset_wheel" value="-${base_len/2 + wheel_radius}" />
+        <xacro:property name="x_offset_front_wheel" value="${base_radius - wheel_radius}" />
+        <xacro:property name="x_offset_back_wheel" value="-${(base_radius - wheel_radius)/2}" />
+        <xacro:property name="y_offset_front_wheel" value="0.00" />
+        <xacro:property name="y_offset_back_wheel" value="${(base_radius - wheel_radius)*SQRT_3/2}" />
         <!-- Base Link -->
         <link name="${prefix}base_link">
@@ -27,11 +26,11 @@
                 <origin xyz="0 0 0" rpy="0 0 0"/>
                 <geometry>
-                    <box size="${base_width} ${base_length} ${base_height}"/>
+                    <cylinder length="${base_len}" radius="${base_radius}"/>
                 </geometry>
             </collision>
             <visual>
-                <origin xyz="0 0 ${base_height/2}" rpy="0 0 0"/>
+                <origin xyz="0 0 0" rpy="0 0 0"/>
                 <geometry>
-                    <box size="${base_width} ${base_length} ${base_height}"/>
+                    <cylinder length="${base_len}" radius="${base_radius}"/>
                 </geometry>
                 <material name="orange"/>
@@ -40,11 +39,15 @@
                 <origin xyz="0 0 0" rpy="0 0 0"/>
                 <mass value="${base_mass}"/>
-                <inertia ixx="${base_mass / 12.0 * (base_length*base_length + base_height*base_height)}" ixy="0.0" ixz="0.0" iyy="${base_mass / 12.0 * (base_height*base_height + base_width*base_width)}" iyz="0.0" izz="${base_mass / 12.0 * (base_width*base_width + base_length*base_length)}"/>
+                <inertia ixx="${base_mass / 12.0 * (3*base_radius*base_radius + base_len*base_len)}" ixy="0.0" ixz="0.0" iyy="${base_mass / 12.0 * (3*base_radius*base_radius + base_len*base_len)}" iyz="0.0" izz="${base_mass / 2.0 * base_radius*base_radius}"/>
             </inertial>
         </link>
+        <!-- Foot Print -->
+        <link name="${prefix}base_footprint"/>
+        <!-- left wheel center Link -->
+        <link name="${prefix}left_wheel_center"/>
         <!-- left wheel Link -->
         <link name="${prefix}left_wheel">
             <collision>
-                <origin xyz="0 0 0" rpy="${PI/2} 0 0"/>
+                <origin xyz="0 0 0" rpy="0 0 0"/>
                 <geometry>
                     <cylinder length="${wheel_len}" radius="${wheel_radius}"/>
@@ -52,20 +55,22 @@
             </collision>
             <visual>
-                <origin xyz="0 0 0" rpy="${PI/2} 0 0"/>
+                <origin xyz="0 0 0" rpy="0 0 0"/>
                 <geometry>
                     <cylinder length="${wheel_len}" radius="${wheel_radius}"/>
                 </geometry>
-                <material name="black"/>
+                <material name="brown"/>
             </visual>
             <inertial>
-                <origin xyz="0 0 0" rpy="${PI/2} 0 0"/>
+                <origin xyz="0 0 0" rpy="0 0 0"/>
                 <mass value="${wheel_mass}"/>
                 <inertia ixx="${wheel_mass / 12.0 * (3*wheel_radius*wheel_radius + wheel_len*wheel_len)}" ixy="0.0" ixz="0.0" iyy="${wheel_mass / 12.0 * (3*wheel_radius*wheel_radius + wheel_len*wheel_len)}" iyz="0.0" izz="${wheel_mass / 2.0 * wheel_radius*wheel_radius}"/>
             </inertial>
         </link>
+        <!-- right wheel center Link -->
+        <link name="${prefix}right_wheel_center"/>
         <!-- right wheel Link -->
         <link name="${prefix}right_wheel">
             <collision>
-                <origin xyz="0 0 0" rpy="${PI/2} 0 0"/>
+                <origin xyz="0 0 0" rpy="0 0 0"/>
                 <geometry>
                     <cylinder length="${wheel_len}" radius="${wheel_radius}"/>
@@ -73,12 +78,12 @@
             </collision>
             <visual>
-                <origin xyz="0 0 0" rpy="${PI/2} 0 0"/>
+                <origin xyz="0 0 0" rpy="0 0 0"/>
                 <geometry>
                     <cylinder length="${wheel_len}" radius="${wheel_radius}"/>
                 </geometry>
-                <material name="black"/>
+                <material name="brown"/>
             </visual>
             <inertial>
-                <origin xyz="0 0 0" rpy="${PI/2} 0 0"/>
+                <origin xyz="0 0 0" rpy="0 0 0"/>
                 <mass value="${wheel_mass}"/>
                 <inertia ixx="${wheel_mass / 12.0 * (3*wheel_radius*wheel_radius + wheel_len*wheel_len)}" ixy="0.0" ixz="0.0" iyy="${wheel_mass / 12.0 * (3*wheel_radius*wheel_radius + wheel_len*wheel_len)}" iyz="0.0" izz="${wheel_mass / 2.0 * wheel_radius*wheel_radius}"/>
@@ -90,5 +95,5 @@
                 <origin xyz="0 0 0" rpy="0 0 0"/>
                 <geometry>
-                    <sphere radius="${caster_wheel_radius}"/>
+                    <sphere radius="${wheel_radius}"/>
                 </geometry>
             </collision>
@@ -96,31 +101,41 @@
                 <origin xyz="0 0 0" rpy="0 0 0"/>
                 <geometry>
-                    <sphere radius="${caster_wheel_radius}"/>
+                    <sphere radius="${wheel_radius}"/>
                 </geometry>
-                <material name="white"/>
+                <material name="gray"/>
             </visual>
             <inertial>
                 <origin xyz="0 0 0" rpy="0 0 0"/>
                 <mass value="${caster_wheel_mass}"/>
-                <inertia ixx="${caster_wheel_mass * 0.4 * (caster_wheel_radius * caster_wheel_radius)}" ixy="0.0" ixz="0.0" iyy="${caster_wheel_mass * 0.4 * (caster_wheel_radius * caster_wheel_radius)}" iyz="0.0" izz="${caster_wheel_mass * 0.4 * (caster_wheel_radius * caster_wheel_radius)}"/>
+                <inertia ixx="${caster_wheel_mass * 0.4 * (wheel_radius * wheel_radius)}" ixy="0.0" ixz="0.0" iyy="${caster_wheel_mass * 0.4 * (wheel_radius * wheel_radius)}" iyz="0.0" izz="${caster_wheel_mass * 0.4 * (wheel_radius * wheel_radius)}"/>
             </inertial>
         </link>
         <joint name="${prefix}base_link_joint" type="fixed">
-            <parent link="${prefix}base_footprint"/>
-            <child link="${prefix}base_link"/>
-            <origin xyz="0 0 ${wheel_radius - z_offset}" rpy="0 0 0"/>
+            <parent link="${prefix}base_link"/>
+            <child link="${prefix}base_footprint"/>
+            <origin xyz="${x_offset_back_wheel} 0 ${z_offset_wheel - wheel_radius}" rpy="0 0 0"/>
+        </joint>
+        <joint name="${prefix}left_wheel_center_joint" type="fixed">
+            <parent link="${prefix}base_link"/>
+            <child link="${prefix}left_wheel_center"/>
+            <origin xyz="${x_offset_back_wheel} ${y_offset_back_wheel} ${z_offset_wheel}" rpy="-${PI/2} 0 0"/>
         </joint>
         <joint name="${prefix}left_wheel_joint" type="continuous">
-            <parent link="${prefix}base_link"/>
+            <parent link="${prefix}left_wheel_center"/>
             <child link="${prefix}left_wheel"/>
-            <origin xyz="${x_offset_tail} -${base_width/2} ${z_offset}" rpy="0 0 0"/>
-            <axis xyz="0 1 0"/>
+            <origin xyz="0 0 0" rpy="0 0 0"/>
+            <axis xyz="0 0 1"/>
             <dynamics damping="0.2"/>
         </joint>
+        <joint name="${prefix}right_wheel_center_joint" type="fixed">
+            <parent link="${prefix}base_link"/>
+            <child link="${prefix}right_wheel_center"/>
+            <origin xyz="${x_offset_back_wheel} -${y_offset_back_wheel} ${z_offset_wheel}" rpy="-${PI/2} 0 0"/>
+        </joint>
         <joint name="${prefix}right_wheel_joint" type="continuous">
-            <parent link="${prefix}base_link"/>
+            <parent link="${prefix}right_wheel_center"/>
             <child link="${prefix}right_wheel"/>
-            <origin xyz="${x_offset_tail} ${base_width/2} ${z_offset}" rpy="0 0 0"/>
-            <axis xyz="0 1 0"/>
+            <origin xyz="0 0 0" rpy="0 0 0"/>
+            <axis xyz="0 0 1"/>
             <dynamics damping="0.2"/>
         </joint>
@@ -128,5 +143,5 @@
             <parent link="${prefix}base_link"/>
             <child link="${prefix}caster_frontal_wheel"/>
-            <origin xyz="${x_offset_head} 0 ${z_offset}" rpy="0 0 0"/>
+            <origin xyz="${x_offset_front_wheel} ${y_offset_front_wheel} ${z_offset_wheel}" rpy="0 0 0"/>
         </joint>
     </xacro:macro>
